File: Acquisition/Schematics/ADC_MainBoard/ADC_MainBoard.kicad_sch (KiCad schematic)
At the start: 49 parts, among them J1 Conn_02x06_Counter_Clockwise, J13 Conn_01x02_Pin, J14 Pad, J15 Pad, J16 Pad, J17 Pad, J2 Pad, J3 Pad, J5 2004850720, J6 Conn_02x06_Counter_Clockwise, J7 Pad, J8 Pad, J9 Pad, U1 MCP1525-TT, U3 OPA333xxDBV, U5 LP5907MFX-2.8, U6 LP5907MFX-1.2, U7 LD1117S33TR_SOT223

Commit message: Schematics - FPGA board seems done
Parts:
- removed C2: 100n, Capacitor_SMD:C_0603_1608Metric, symbol Device:C
- removed R2: 1K, Capacitor_SMD:C_0603_1608Metric, symbol Device:R
- added C12, C13, C14, C15: 100n, Capacitor_SMD:C_0603_1608Metric, symbol Device:C
- added C16, C17: 4.7u, Capacitor_SMD:C_0603_1608Metric, symbol Device:C
- added C18: 470n, Capacitor_SMD:C_0603_1608Metric, symbol Device:C
- added FB1: FerriteBead, Capacitor_THT:CP_Axial_L11.0mm_D6.0mm_P18.00mm_Horizontal, symbol Device:FerriteBead
- added J4: Conn_02x12_Odd_Even, Connector_PinHeader_2.54mm:PinHeader_2x12_P2.54mm_Vertical, symbol Connector_Generic:Conn_02x12_Odd_Even
- added R20, R21: 0, Resistor_SMD:R_0603_1608Metric, symbol Device:R
- added R22: 33.2k, Resistor_SMD:R_0603_1608Metric, symbol Device:R
- added U4: TPS7A2033, Package_TO_SOT_SMD:SOT-23-5, symbol Regulator_Linear:LP5907MFX-2.8
- added U8: LT3042xMSE, Package_SO:MSOP-10-1EP_3x3mm_P0.5mm_EP1.68x1.88mm, symbol Regulator_Linear:LT3042xMSE
- R1: value 1K -> 0
Connections:
- net +3.3V: now also J1.6 (Pin_6), C12.1; no longer J1.12 (Pin_12), U1.1 (Vin), U3.5 (V+)
- net +5V: now also FB1.1; no longer C8.1, U5.1 (IN), U5.3 (EN)
- net CamVSYNC: now also J4.15 (Pin_15)
- net Earth: now also J1.11 (Pin_11), C12.2, J4.1 (Pin_1), J4.12 (Pin_12), J4.17 (Pin_17), J4.21 (Pin_21), J4.5 (Pin_5), J4.9 (Pin_9); no longer C1.2, C7.2, J1.6 (Pin_6), J1.9 (Pin_9), J6.3 (Pin_3), J6.6 (Pin_6), J6.9 (Pin_9), R1.1, U1.3 (Vss), U2.23 (AGND), U3.2 (V-)
- net PCLK: no longer C5.1, U2.8 (PCLK)
- net REFIN+: now also R1.2
- net nCS: now also J1.9 (Pin_9); no longer J1.10 (Pin_10)
- net nIRQ: now also J1.10 (Pin_10); no longer J1.11 (Pin_11)
- net nIRQ___2: no longer J6.11 (Pin_11)
- net at C1.1, R3.1, U1.2 (Vout): now also R1.1
- net REFIN- renamed AVdd
- net AVdd: now also C15.2, R20.1, R21.1; no longer R4.1
- new net: C18.1, R22.1, U8.7 (SET)
- new net +3.3VA: C14.1, C17.1, R20.2, U1.1 (Vin), U3.5 (V+), U4.5 (OUT), U8.10 (OUT), U8.9 (OUTS)
- new net +5VA: C13.1, C16.1, C8.1, FB1.2, R21.2, U4.1 (IN), U4.3 (EN), U5.1 (IN), U5.3 (EN), U8.1 (IN), U8.2 (IN), U8.3 (EN/UV), U8.6 (PGFB)
- new net 5v: J4.2 (Pin_2)
- new net CONVST: J4.4 (Pin_4)
- new net CamPCLK: C5.1, J4.16 (Pin_16), U2.8 (PCLK)
- new net GND: C1.2, C13.2, C14.2, C15.1, C16.2, C17.2, C18.2, C7.2, J1.12 (Pin_12), J6.3 (Pin_3), J6.6 (Pin_6), J6.9 (Pin_9), R22.2, R4.1, U1.3 (Vss), U2.23 (AGND), U3.2 (V-), U4.2 (GND), U8.11 (GND), U8.5 (ILIM), U8.8 (GND)
- new net MISO11: J4.18 (Pin_18)
- new net MISO12: J4.20 (Pin_20)
- new net MISO13: J4.22 (Pin_22)
- new net MISO14: J4.24 (Pin_24)
- new net MISO2: J4.14 (Pin_14)
- new net MISO3: J4.11 (Pin_11)
- new net MISO4: J4.7 (Pin_7)
- new net MISO5: J4.19 (Pin_19)
- new net MISO6: J4.23 (Pin_23)
- new net MISO7: J4.8 (Pin_8)
- new net MISO8: J4.10 (Pin_10)
- new net MISO9: J4.13 (Pin_13)
- new net MOSI: J4.6 (Pin_6)
- new net SCLK: J4.3 (Pin_3)
Other:
- moved on the sheet: J13, J14, J15, J16, J17, J7, J8, J9

Commit message: Acquisition schematics should be working.
Parts:
- removed C15: 100n, Capacitor_SMD:C_0603_1608Metric, symbol Device:C
- removed J2, J3, J8, J9: Pad, CustomLibrary:Pad, symbol Connector:Conn_01x01_Pin
- removed J6: Conn_02x06_Counter_Clockwise, CustomLibrary:KYOCERA AVX Base, symbol Connector_Generic:Conn_02x06_Counter_Clockwise
- removed R11, R12, R13, R14, R15, R16, R17, R18, R19: 10, Capacitor_SMD:C_0603_1608Metric, symbol Device:R
- removed R20, R21: 0, Resistor_SMD:R_0603_1608Metric, symbol Device:R
- added J10: 2004850720, CustomLibrary:Molex FFC 20pin sideways, symbol 2026-01-08_16-40-01:2004850720
- added J11, J12, J18, J19, J20, J21, J22, J23, J24, J25, J26, J27, J28, J29, J30: ADC_Conn, CustomLibrary:KYOCERA AVX Base, symbol Connector_Generic:Conn_02x06_Counter_Clockwise
- J1: value Conn_02x06_Counter_Clockwise -> ADC_Conn
- J5: footprint CON_2004850720 -> CustomLibrary:Molex FFC 20pin sideways
Connections:
- net 5v is gone; now on net +5V: J4.2 (Pin_2)
- net AVdd is gone; now on net +3.3VA: J1.1 (Pin_1)
- net CONVST is gone; now on net CamD4: J4.4 (Pin_4)
- net MISO11 is gone; now on net CamD2: J4.18 (Pin_18)
- net MISO12 is gone; now on net CamD6: J4.20 (Pin_20)
- net MISO13 is gone; now on net CamSCK: J4.22 (Pin_22)
- net MISO2 is gone; now on net CamHSYNC: J4.14 (Pin_14)
- net MISO3 is gone; now on net CamD5: J4.11 (Pin_11)
- net MISO4 is gone; now on net CamD1: J4.7 (Pin_7)
- net MISO5 is gone; now on net CamRST: J4.19 (Pin_19)
- net MISO6 is gone; now on net CamSDA: J4.23 (Pin_23)
- net MISO7 is gone; now on net CamMCLK: J4.8 (Pin_8)
- net MISO8 is gone; now on net CamD7: J4.10 (Pin_10)
- net MISO9 is gone; now on net CamPWDN: J4.13 (Pin_13)
- net MOSI is gone; now on net CamD3: J4.6 (Pin_6)
- net SCLK is gone; now on net CamD0: J4.3 (Pin_3)
- net nIRQ is gone; now on net Earth: J1.10 (Pin_10)
- net nIRQ___2 is gone; now on net nCS: J5.20
- net nIRQ___3 is gone; now on net MCLK: J5.19
- net +3.3V: now also J11.6 (Pin_6), J12.6 (Pin_6), J18.6 (Pin_6), J19.6 (Pin_6), J20.6 (Pin_6), J21.6 (Pin_6), J22.6 (Pin_6), J23.6 (Pin_6), J24.6 (Pin_6), J25.6 (Pin_6), J26.6 (Pin_6), J27.6 (Pin_6), J28.6 (Pin_6), J29.6 (Pin_6), J30.6 (Pin_6)
- net +3.3VA: now also J11.1 (Pin_1), J12.1 (Pin_1), J18.1 (Pin_1), J19.1 (Pin_1), J20.1 (Pin_1), J21.1 (Pin_1), J22.1 (Pin_1), J23.1 (Pin_1), J24.1 (Pin_1), J25.1 (Pin_1), J26.1 (Pin_1), J27.1 (Pin_1), J28.1 (Pin_1), J29.1 (Pin_1), J30.1 (Pin_1)
- net +5VA: now also J1.2 (Pin_2), J11.2 (Pin_2), J12.2 (Pin_2), J18.2 (Pin_2), J19.2 (Pin_2), J20.2 (Pin_2), J21.2 (Pin_2), J22.2 (Pin_2), J23.2 (Pin_2), J24.2 (Pin_2), J25.2 (Pin_2), J26.2 (Pin_2), J27.2 (Pin_2), J28.2 (Pin_2), J29.2 (Pin_2), J30.2 (Pin_2)
- net CamD3: no longer J5.10
- net CamD6: no longer J5.12
- net CamD7: no longer J5.14
- net CamHSYNC: no longer J5.15
- net CamMCLK: no longer J5.13
- net CamPCLK: now also J16.1 (Pin_1)
- net CamSCK: no longer J5.17
- net CamSDA: no longer J5.18
- net CamVSYNC: no longer J5.16
- net Earth: now also C7.2, J10.G1, J10.G2, J10.P1, J10.P2, J10.P3, J10.P4, J11.10 (Pin_10), J11.3 (Pin_3), J12.10 (Pin_10), J12.3 (Pin_3), J18.10 (Pin_10), J18.3 (Pin_3), J19.10 (Pin_10), J19.3 (Pin_3), J20.10 (Pin_10), J20.3 (Pin_3), J21.10 (Pin_10), J21.3 (Pin_3), J22.10 (Pin_10), J22.3 (Pin_3), J23.10 (Pin_10), J23.3 (Pin_3), J24.10 (Pin_10), J24.3 (Pin_3), J25.10 (Pin_10), J25.3 (Pin_3), J26.10 (Pin_10), J26.3 (Pin_3), J27.10 (Pin_10), J27.3 (Pin_3), J28.10 (Pin_10), J28.3 (Pin_3), J29.10 (Pin_10), J29.3 (Pin_3), J30.10 (Pin_10), J30.3 (Pin_3); no longer C8.2, C9.2, J1.11 (Pin_11), U5.2 (GND)
- net GND: now also C8.2, C9.2, U5.2 (GND), J11.12 (Pin_12), J12.12 (Pin_12), J18.12 (Pin_12), J19.12 (Pin_12), J20.12 (Pin_12), J21.12 (Pin_12), J22.12 (Pin_12), J23.12 (Pin_12), J24.12 (Pin_12), J25.12 (Pin_12), J26.12 (Pin_12), J27.12 (Pin_12), J28.12 (Pin_12), J29.12 (Pin_12), J30.12 (Pin_12); no longer C7.2
- net MCLK: now also J10.19, J11.7 (Pin_7), J12.7 (Pin_7), J18.7 (Pin_7), J19.7 (Pin_7), J20.7 (Pin_7), J21.7 (Pin_7), J22.7 (Pin_7), J23.7 (Pin_7), J24.7 (Pin_7), J25.7 (Pin_7), J26.7 (Pin_7), J27.7 (Pin_7), J28.7 (Pin_7), J29.7 (Pin_7), J30.7 (Pin_7)
- net REFIN+: now also J1.11 (Pin_11), J11.11 (Pin_11), J12.11 (Pin_11), J18.11 (Pin_11), J19.11 (Pin_11), J20.11 (Pin_11), J21.11 (Pin_11), J22.11 (Pin_11), J23.11 (Pin_11), J24.11 (Pin_11), J25.11 (Pin_11), J26.11 (Pin_11), J27.11 (Pin_11), J28.11 (Pin_11), J29.11 (Pin_11), J30.11 (Pin_11); no longer J1.2 (Pin_2)
- net SCK: now also J5.18, J10.18, J11.4 (Pin_4), J12.4 (Pin_4), J18.4 (Pin_4), J19.4 (Pin_4), J20.4 (Pin_4), J21.4 (Pin_4), J22.4 (Pin_4), J23.4 (Pin_4), J24.4 (Pin_4), J25.4 (Pin_4), J26.4 (Pin_4), J27.4 (Pin_4), J28.4 (Pin_4), J29.4 (Pin_4), J30.4 (Pin_4)
- net SDI: now also J5.17, J10.17, J11.5 (Pin_5), J12.5 (Pin_5), J18.5 (Pin_5), J19.5 (Pin_5), J20.5 (Pin_5), J21.5 (Pin_5), J22.5 (Pin_5), J23.5 (Pin_5), J24.5 (Pin_5), J25.5 (Pin_5), J26.5 (Pin_5), J27.5 (Pin_5), J28.5 (Pin_5), J29.5 (Pin_5), J30.5 (Pin_5)
- net nCS: now also J10.20, J11.9 (Pin_9), J12.9 (Pin_9), J18.9 (Pin_9), J19.9 (Pin_9), J20.9 (Pin_9), J21.9 (Pin_9), J22.9 (Pin_9), J23.9 (Pin_9), J24.9 (Pin_9), J25.9 (Pin_9), J26.9 (Pin_9), J27.9 (Pin_9), J28.9 (Pin_9), J29.9 (Pin_9), J30.9 (Pin_9)
- net SDO19: now reaches J5.1
- net SDO19: now also J10.5, J24.8 (Pin_8)
- net CamPWDN: now reaches R8.1, U2.17 (PWDN)
- net SDO1A: now reaches J5.3
- net SDO1A: now also J10.7, J25.8 (Pin_8)
- net SDO15: now reaches J5.6
- net SDO15: now also J10.4, J20.8 (Pin_8)
- net SDO14: now reaches J5.8
- net SDO14: now also J10.2, J19.8 (Pin_8)
- net SDO1B: now reaches J5.5
- net SDO1B: now also J10.16, J26.8 (Pin_8)
- net SDO16: now reaches J5.2
- net SDO16: now also J10.6, J21.8 (Pin_8)
- net SDO10: now reaches J5.4
- net SDO10: now also J1.8 (Pin_8), J10.10
- net SDO18: now reaches J5.7
- net SDO18: now also J10.3, J23.8 (Pin_8)
- net SDO17: now reaches J5.9
- net SDO17: now also J10.1, J22.8 (Pin_8)
- net PCLK renamed SDO1F
- net SDO1F: now also J10.9, J30.8 (Pin_8)
- removed net SDO1: J1.8 (Pin_8), J16.1 (Pin_1)
- net SDO2 renamed SDO1D
- net SDO1D: now also J5.14, J10.14, J28.8 (Pin_8)
- new net SDO11: J10.12, J11.8 (Pin_8), J5.16
- new net SDO12: J10.11, J12.8 (Pin_8), J5.12
- new net SDO13: J10.8, J18.8 (Pin_8), J5.10
- new net SDO1C: J10.15, J27.8 (Pin_8), J5.13
- new net SDO1E: J10.13, J29.8 (Pin_8), J5.15
Other:
- moved on the sheet: C13, C14, C16, C17, C18, J4, R22, U4, U8
