File: Acquisition/Schematics/ADC_MainBoard/_autosave-ADC_MainBoard.kicad_sch (KiCad schematic)
At the start: 60 parts, among them J1 ADC_Conn, J10 2004850720, J11 ADC_Conn, J12 ADC_Conn, J13 Conn_01x02_Pin, J14 Pad, J15 Pad, J16 Pad, J17 Pad, J18 ADC_Conn, J19 ADC_Conn, J20 ADC_Conn, J21 ADC_Conn, J22 ADC_Conn, J23 ADC_Conn, J24 ADC_Conn, J25 ADC_Conn, J26 ADC_Conn, J27 ADC_Conn, J28 ADC_Conn, J29 ADC_Conn, J30 ADC_Conn, J4 Conn_02x12_Odd_Even, J5 2004850720, J7 Pad, U1 MCP1525-TT, U3 OPA333xxDBV, U4 TPS7A2033, U5 LP5907MFX-2.8, U6 LP5907MFX-1.2, U7 LD1117S33TR_SOT223, U8 LT3042xMSE

Commit message: PCBs production ready
Parts:
- added C2: 100n, Capacitor_Tantalum_SMD:CP_EIA-3528-21_Kemet-B, symbol Device:C
Connections:
- net +5VA: now also C2.1
- net GND: now also C2.2
Changed lines of the file:
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@@
   (junction (at 217.17 144.78) (diameter 0) (color 0 0 0 0)
+  )
+  (junction (at 162.56 160.02) (diameter 0) (color 0 0 0 0)
   )
   (wire (pts (xy 106.68 100.33) (xy 114.3 100.33))
@@
         (path "/89c9ff72-9916-4865-897e-a40a0c4dfe2f"
           (reference "#PWR011") (unit 1)
+        )
+      )
+    )
+  )
+  (symbol (lib_id "power:GND") (at 162.56 167.64 0) (unit 1)
+    (in_bom yes) (on_board yes) (dnp no) (fields_autoplaced)
+    (property "Reference" "#PWR09" (at 162.56 173.99 0)
+      (effects (font (size 1.27 1.27)) hide)
+    )
+    (property "Value" "GND" (at 162.56 172.72 0)
+      (effects (font (size 1.27 1.27)))
+    )
+    (property "Footprint" "" (at 162.56 167.64 0)
+      (effects (font (size 1.27 1.27)) hide)
+    )
+    (property "Datasheet" "" (at 162.56 167.64 0)
+      (effects (font (size 1.27 1.27)) hide)
+    )
+    (pin "1")
+    (instances
+      (project "ADC_MainBoard"
+        (path "/89c9ff72-9916-4865-897e-a40a0c4dfe2f"
+          (reference "#PWR09") (unit 1)
         )
       )
@@
         )
       )
+    )
+  )
+  (symbol (lib_id "Device:C") (at 162.56 163.83 0) (unit 1)
+    (in_bom yes) (on_board yes) (dnp no)
+    (property "Reference" "C2" (at 161.29 156.21 0)
+      (effects (font (size 1.27 1.27)) (justify left))
+    )
+    (property "Value" "100n" (at 161.29 158.75 0)
+      (effects (font (size 1.27 1.27)) (justify left))
+    )
+    (property "Footprint" "Capacitor_Tantalum_SMD:CP_EIA-3528-21_Kemet-B" (at 163.5252 167.64 0)
+      (effects (font (size 1.27 1.27)) hide)
+    )
+    (property "Datasheet" "~" (at 162.56 163.83 0)
+      (effects (font (size 1.27 1.27)) hide)
+    )
+    (pin "2")
+    (pin "1")
+    (instances
+      (project "ADC_MainBoard"
+        (path "/89c9ff72-9916-4865-897e-a40a0c4dfe2f"
+          (reference "C2") (unit 1)
+        )
+      )
