File: Acquisition/Schematics/Locator_FPGA/mic_array.kicad_sch (KiCad schematic)
At the start: 59 parts, among them J1 Conn_02x07_Odd_Even, J3 Conn_02x12_Odd_Even, J4 2004850720, J8 2004850720, U1 XC6SLX9-TQG144, U2 M25PX32-VMW, U9 M95256-WMN6P, X1 XO91

Commit message: Schematics - FPGA board seems done
Parts:
- added R29, R33: 30, Resistor_SMD:R_0603_1608Metric, symbol Device:R
- added RN1, RN2, RN3: R_Pack04, Resistor_SMD:R_Array_Concave_4x0402, symbol Device:R_Pack04
- added U3: M95256-WMN6P, Package_SO:SOIC-8_3.9x4.9mm_P1.27mm, symbol Memory_EEPROM:M95256-WMN6P
- R24, R25: value 0 -> 30
Connections:
- net ADC_PAR10 is gone; now on net ADC_PAR5: U1.141 (IO_L2N_0)
- net ADC_PAR11 is gone; now on net ADC_PAR6: U1.140 (IO_L3P_0)
- net ADC_PAR12 is gone; now on net ADC_PAR7: U1.139 (IO_L3N_0)
- net ADC_PAR4 is gone; now on net SW5: U1.115 (IO_L65P_SCP3_0)
- net ADC_PAR8 is gone; now on net FFC2_19: U1.119 (IO_L63P_SCP7_0)
- net 3v3: now also U3.8 (VCC)
- net ADC_PAR5: no longer U1.116 (IO_L64N_SCP4_0)
- net ADC_PAR6: no longer U1.117 (IO_L64P_SCP5_0)
- net ADC_PAR7: no longer U1.118 (IO_L63N_SCP6_0)
- net EEPROM_C: now also R29.2; no longer U9.6 (C)
- net EEPROM_D: now also RN2.8 (R1.2); no longer U9.5 (D)
- net EEPROM_Q: now also RN2.6 (R3.2); no longer U9.2 (Q)
- net EEPROM_nH: now also R25.1; no longer U9.7 (~{HOLD})
- net EEPROM_nS: now also RN2.5 (R4.2); no longer U9.1 (~{S})
- net EEPROM_nW: now also RN2.7 (R2.2); no longer U9.3 (~{W})
- net Earth: now also U3.4 (VSS)
- net FFC2_19: no longer U1.120 (IO_L62N_VREF_0)
- net FFC2_20: now also U1.120 (IO_L62N_VREF_0); no longer U1.126 (IO_L36N_GCLK14_0)
- net SW4: now also U1.116 (IO_L64N_SCP4_0); no longer U1.93 (IO_L41P_GCLK9_IRDY1_1)
- net SW5: no longer U1.94 (IO_L40N_GCLK10_1)
- net ADC_BSY renamed FSMC_DA1
- net ADC_CLK renamed FSMC_NWE
- net ADC_DIN renamed FSMC_NWAIT
- net ADC_PAR1 renamed FSMC_DA2
- net ADC_PAR13 renamed EEPROM2_nW
- net EEPROM2_nW: now also RN1.1 (R1.1)
- net ADC_PAR14 renamed EEPROM2_D
- net EEPROM2_D: now also RN1.2 (R2.1)
- net ADC_PAR15 renamed EEPROM2_C
- net EEPROM2_C: now also RN1.3 (R3.1)
- net ADC_PAR16 renamed EEPROM2_Q
- net EEPROM2_Q: now also RN1.4 (R4.1)
- net ADC_PAR2 renamed FSMC_DA3
- net ADC_PAR3 renamed FSMC_NL
- net ADC_PAR9 renamed FSMC_DA4
- net Additional_1 renamed EEPROM2_nS
- net EEPROM2_nS: now also R33.1
- net Additional_2 renamed EEPROM2_nH
- net EEPROM2_nH: now also R24.1
- net CONVST renamed CamRST
- net CamRST: no longer R24.1
- net FFC2_21 renamed ADC_SDI
- net ADC_SDI: now also J8.4, RN3.8 (R1.2); no longer U1.127 (IO_L36P_GCLK15_0)
- net FFC2_22: no longer names the net of R24.2
- net FFC2_22: now also U3.7 (~{HOLD}); no longer J4.18
- net FFC2_23: no longer names the net of R25.2
- net FFC2_23: now also U9.5 (D); no longer J4.19
- net FFC3_06: no longer names the net of U1.48 (IO_L48P_D7_2)
- net FFC3_06: now also RN3.4 (R4.1); no longer J8.2
- net FFC3_07: no longer names the net of U1.50 (IO_L31N_GCLK30_D15_2)
- net FFC3_07: now also RN3.3 (R3.1); no longer J8.3
- net FFC3_08: no longer names the net of U1.51 (IO_L31P_GCLK31_D14_2)
- net FFC3_08: now also RN3.1 (R1.1); no longer J8.4
- net MISO1 renamed CamVSYNC
- net MISO10 renamed CamPCLK
- net MISO11 renamed CamD4
- net MISO12 renamed CamD0
- net MISO13 renamed CamD1
- net MISO2 renamed CamD6
- net MISO3 renamed CamMCLK
- net MISO4 renamed CamHSYNC
- net MISO5 renamed CamD2
- net MISO6 renamed CamD3
- net MISO7 renamed CamSDA
- net MISO8 renamed CamD7
- net MISO9 renamed CamD5
- net CamD5: now also U1.93 (IO_L41P_GCLK9_IRDY1_1); no longer U1.95 (IO_L40P_GCLK11_1)
- net MOSI renamed CamSCK
- net SCLK renamed CamPWDN
- net CamPWDN: no longer R25.1
- new net: R33.2, U3.1 (~{S})
- new net: R29.1, U9.6 (C)
- new net: RN1.5 (R4.2), U3.2 (Q)
- new net: RN1.6 (R3.2), U3.6 (C)
- new net: RN1.7 (R2.2), U3.5 (D)
- new net: RN1.8 (R1.2), U3.3 (~{W})
- new net: RN2.2 (R2.1), U9.1 (~{S})
- new net: RN2.3 (R3.1), U9.2 (Q)
- new net: RN2.4 (R4.1), U9.3 (~{W})
- new net: RN2.1 (R1.1), U9.7 (~{HOLD})
- new net ADC_MCLK: J4.19, J8.2, RN3.5 (R4.2)
- new net ADC_SCK: J4.18, J8.3, RN3.6 (R3.2)
- new net FSMC_CLK: U1.95 (IO_L40P_GCLK11_1)
- new net FSMC_DA0: U1.126 (IO_L36N_GCLK14_0)
- new net FSMC_NE1: U1.127 (IO_L36P_GCLK15_0)
- new net FSMC_NOE: U1.94 (IO_L40N_GCLK10_1)
- new net STATUS: U1.117 (IO_L64P_SCP5_0)
Other:
- moved on the sheet: J3

Commit message: Acquisition schematics should be working.
Parts:
- J4, J8: footprint CON_2004850720 -> CustomLibrary:Molex FFC 20pin sideways
Changed lines of the file:
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@@
       (effects (font (size 1.524 1.524)) (justify left))
     )
-    (property "Footprint" "CON_2004850720" (at -20.32 3.81 0)
+    (property "Footprint" "CustomLibrary:Molex FFC 20pin sideways" (at -20.32 3.81 0)
       (effects (font (size 1.27 1.27) italic) hide)
     )
@@
       (effects (font (size 1.524 1.524)) (justify left))
     )
-    (property "Footprint" "CON_2004850720" (at 27.94 5.08 0)
+    (property "Footprint" "CustomLibrary:Molex FFC 20pin sideways" (at 27.94 5.08 0)
       (effects (font (size 1.27 1.27) italic) hide)
     )
