File: Acquisition/Schematics/Locator_FPGA/Locator_FPGA.kicad_sch (KiCad schematic)
At the start: 79 parts, among them J2 USB_A, J5 Conn_02x03_Odd_Even, J6 OUTPUT Barrel, J7 Conn_01x02, Q1 IRLML9301, SW1 SW_DIP_x08, U4 USB3300-EZK, U6 STM32F407VETx, U7 AMS1117, U8 AMS1117, Y1 Crystal, Y2 Crystal_GND24

Commit message: Schematics - FPGA board seems done
Parts:
- removed D7: LED, LED_SMD:LED_0805_2012Metric, symbol Device:LED
- removed R29: 200R, Resistor_SMD:R_0603_1608Metric, symbol Device:R
- J6: footprint Connector_BarrelJack:BarrelJack_Horizontal -> Connector_PinHeader_2.54mm:PinHeader_1x02_P2.54mm_Vertical
Connections:
- net ADC_BSY: no longer U6.65 (PC8)
- net ADC_CLK: no longer U6.67 (PA8)
- net Earth: no longer U6.38 (PE7), U6.39 (PE8), U6.40 (PE9), U6.41 (PE10)
- net STATUS: now reaches U6.69 (PA10)
- net ADC_CS2 renamed DONE
- net ADC_DIN renamed MOSI_1
- net ADC_PAR_D1 renamed FSMC_DA2
- net ADC_PAR_D15 renamed FSMC_DA0
- net ADC_PAR_D16 renamed FSMC_DA1
- net ADC_PAR_D2 renamed FSMC_DA3
- net ADC_PAR_D3: no longer names the net of U6.83 (PD2)
- net ADC_PAR_D4 renamed FSMC_CLK
- net ADC_PAR_D5 renamed FSMC_NOE
- net ADC_PAR_D6 renamed FSMC_NWE
- net ADC_PAR_D7 renamed FSMC_NWAIT
- net ADC_PAR_D8 renamed FSMC_NE1
- net FPGA_additional_1: no longer names the net of U6.64 (PC7)
- net FPGA_additional_2: no longer names the net of U6.63 (PC6)
- net LED6 renamed FSMC_NL
- new net FSMC_DA4: U6.38 (PE7)
- new net FSMC_DA5: U6.39 (PE8)
- new net FSMC_DA6: U6.40 (PE9)
- new net FSMC_DA7: U6.41 (PE10)
Other:
- sheet MicArray ports: added DONE, FSMC_CLK, FSMC_DA0, FSMC_DA1, FSMC_DA2, FSMC_DA3, FSMC_DA4, FSMC_NE1, FSMC_NL, FSMC_NOE, FSMC_NWAIT, FSMC_NWE, STATUS; removed ADC_BSY, ADC_CLK, ADC_DIN, ADC_PAR1, ADC_PAR10, ADC_PAR11, ADC_PAR12, ADC_PAR15, ADC_PAR16, ADC_PAR2, ADC_PAR3, ADC_PAR4, ADC_PAR8, ADC_PAR9, Additional_1, Additional_2

Commit message: PCBs production ready
Parts:
- added J10, J11, J12, J13, J14, J9: Pad, CustomLibrary:Pad, symbol Connector:Conn_01x01_Pin
Connections:
- net FSMC_CLK: now also J10.1 (Pin_1)
- net FSMC_NE1: now also J14.1 (Pin_1)
- net FSMC_NL: now also J9.1 (Pin_1)
- net FSMC_NOE: now also J12.1 (Pin_1)
- net FSMC_NWAIT: now also J11.1 (Pin_1)
- net FSMC_NWE: now also J13.1 (Pin_1)
Changed lines of the file:
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@@
+    (effects (font (size 1.27 1.27)) (justify left bottom))
+  )
+  (label "FSMC_NOE" (at 123.19 78.74 0) (fields_autoplaced)
     (effects (font (size 1.27 1.27)) (justify left bottom))
   )
@@
     (effects (font (size 1.27 1.27)) (justify left bottom))
   )
+  (label "FSMC_CLK" (at 147.32 83.82 0) (fields_autoplaced)
+    (effects (font (size 1.27 1.27)) (justify left bottom))
+  )
   (label "FSMC_NE1" (at 182.88 109.22 0) (fields_autoplaced)
     (effects (font (size 1.27 1.27)) (justify left bottom))
@@
     (effects (font (size 1.27 1.27)) (justify left bottom))
   )
+  (label "FSMC_NL" (at 147.32 78.74 0) (fields_autoplaced)
+    (effects (font (size 1.27 1.27)) (justify left bottom))
+  )
   (label "ADC_PAR_D10" (at 182.88 114.3 0) (fields_autoplaced)
     (effects (font (size 1.27 1.27)) (justify left bottom))
@@
     (effects (font (size 1.27 1.27)) (justify left bottom))
   )
+  (label "FSMC_NWAIT" (at 147.32 88.9 0) (fields_autoplaced)
+    (effects (font (size 1.27 1.27)) (justify left bottom))
+  )
   (label "USB_DP" (at 241.3 55.88 0) (fields_autoplaced)
     (effects (font (size 1.27 1.27)) (justify left bottom))
@@
   )
   (label "USB_CLK" (at 241.3 134.62 0) (fields_autoplaced)
+    (effects (font (size 1.27 1.27)) (justify left bottom))
+  )
+  (label "FSMC_NWE" (at 123.19 83.82 0) (fields_autoplaced)
     (effects (font (size 1.27 1.27)) (justify left bottom))
   )
@@
   )
   (label "LED3" (at 36.83 168.91 0) (fields_autoplaced)
+    (effects (font (size 1.27 1.27)) (justify left bottom))
+  )
+  (label "FSMC_NE1" (at 123.19 90.17 0) (fields_autoplaced)
     (effects (font (size 1.27 1.27)) (justify left bottom))
   )
@@
     )
   )
+  (symbol (lib_id "Connector:Conn_01x01_Pin") (at 142.24 83.82 0) (unit 1)
+    (in_bom yes) (on_board yes) (dnp no) (fields_autoplaced)
+    (property "Reference" "J10" (at 142.875 78.74 0)
+      (effects (font (size 1.27 1.27)))
+    )
+    (property "Value" "Pad" (at 142.875 81.28 0)
+      (effects (font (size 1.27 1.27)))
+    )
+    (property "Footprint" "CustomLibrary:Pad" (at 142.24 83.82 0)
+      (effects (font (size 1.27 1.27)) hide)
+    )
+    (property "Datasheet" "~" (at 142.24 83.82 0)
+      (effects (font (size 1.27 1.27)) hide)
+    )
+    (pin "1")
+    (instances
+      (project "Locator_FPGA"
+        (path "/33cb5046-a12e-4461-8dbd-367869bd8ded"
+          (reference "J10") (unit 1)
+        )
+      )
+    )
+  )
   (symbol (lib_id "Device:R") (at 116.84 154.94 270) (unit 1)
     (in_bom yes) (on_board yes) (dnp no)
@@
         (path "/33cb5046-a12e-4461-8dbd-367869bd8ded"
           (reference "J7") (unit 1)
+        )
+      )
+    )
+  )
+  (symbol (lib_id "Connector:Conn_01x01_Pin") (at 142.24 78.74 0) (unit 1)
+    (in_bom yes) (on_board yes) (dnp no) (fields_autoplaced)
+    (property "Reference" "J9" (at 142.875 73.66 0)
+      (effects (font (size 1.27 1.27)))
+    )
+    (property "Value" "Pad" (at 142.875 76.2 0)
+      (effects (font (size 1.27 1.27)))
+    )
+    (property "Footprint" "CustomLibrary:Pad" (at 142.24 78.74 0)
+      (effects (font (size 1.27 1.27)) hide)
+    )
+    (property "Datasheet" "~" (at 142.24 78.74 0)
+      (effects (font (size 1.27 1.27)) hide)
+    )
+    (pin "1")
+    (instances
+      (project "Locator_FPGA"
+        (path "/33cb5046-a12e-4461-8dbd-367869bd8ded"
+          (reference "J9") (unit 1)
         )
       )
@@
     )
   )
+  (symbol (lib_id "Connector:Conn_01x01_Pin") (at 142.24 88.9 0) (unit 1)
+    (in_bom yes) (on_board yes) (dnp no) (fields_autoplaced)
+    (property "Reference" "J11" (at 142.875 83.82 0)
+      (effects (font (size 1.27 1.27)))
+    )
+    (property "Value" "Pad" (at 142.875 86.36 0)
+      (effects (font (size 1.27 1.27)))
+    )
+    (property "Footprint" "CustomLibrary:Pad" (at 142.24 88.9 0)
+      (effects (font (size 1.27 1.27)) hide)
+    )
+    (property "Datasheet" "~" (at 142.24 88.9 0)
+      (effects (font (size 1.27 1.27)) hide)
+    )
+    (pin "1")
+    (instances
+      (project "Locator_FPGA"
+        (path "/33cb5046-a12e-4461-8dbd-367869bd8ded"
+          (reference "J11") (unit 1)
+        )
+      )
+    )
+  )
   (symbol (lib_id "Connector:Conn_01x02_Pin") (at 138.43 53.34 90) (unit 1)
     (in_bom yes) (on_board yes) (dnp no)
@@
     )
   )
+  (symbol (lib_id "Connector:Conn_01x01_Pin") (at 118.11 90.17 0) (unit 1)
+    (in_bom yes) (on_board yes) (dnp no) (fields_autoplaced)
+    (property "Reference" "J14" (at 118.745 85.09 0)
+      (effects (font (size 1.27 1.27)))
+    )
+    (property "Value" "Pad" (at 118.745 87.63 0)
+      (effects (font (size 1.27 1.27)))
+    )
+    (property "Footprint" "CustomLibrary:Pad" (at 118.11 90.17 0)
+      (effects (font (size 1.27 1.27)) hide)
+    )
+    (property "Datasheet" "~" (at 118.11 90.17 0)
+      (effects (font (size 1.27 1.27)) hide)
+    )
+    (pin "1")
+    (instances
+      (project "Locator_FPGA"
+        (path "/33cb5046-a12e-4461-8dbd-367869bd8ded"
+          (reference "J14") (unit 1)
+        )
+      )
+    )
+  )
+  (symbol (lib_id "Connector:Conn_01x01_Pin") (at 118.11 78.74 0) (unit 1)
+    (in_bom yes) (on_board yes) (dnp no) (fields_autoplaced)
+    (property "Reference" "J12" (at 118.745 73.66 0)
+      (effects (font (size 1.27 1.27)))
+    )
+    (property "Value" "Pad" (at 118.745 76.2 0)
+      (effects (font (size 1.27 1.27)))
+    )
+    (property "Footprint" "CustomLibrary:Pad" (at 118.11 78.74 0)
+      (effects (font (size 1.27 1.27)) hide)
+    )
+    (property "Datasheet" "~" (at 118.11 78.74 0)
+      (effects (font (size 1.27 1.27)) hide)
+    )
+    (pin "1")
+    (instances
+      (project "Locator_FPGA"
+        (path "/33cb5046-a12e-4461-8dbd-367869bd8ded"
+          (reference "J12") (unit 1)
+        )
+      )
+    )
+  )
   (symbol (lib_id "Device:R") (at 105.41 146.05 0) (unit 1)
     (in_bom yes) (on_board yes) (dnp no)
@@
         )
       )
+    )
+  )
+  (symbol (lib_id "Connector:Conn_01x01_Pin") (at 118.11 83.82 0) (unit 1)
+    (in_bom yes) (on_board yes) (dnp no) (fields_autoplaced)
+    (property "Reference" "J13" (at 118.745 78.74 0)
+      (effects (font (size 1.27 1.27)))
+    )
+    (property "Value" "Pad" (at 118.745 81.28 0)
+      (effects (font (size 1.27 1.27)))
+    )
+    (property "Footprint" "CustomLibrary:Pad" (at 118.11 83.82 0)
+      (effects (font (size 1.27 1.27)) hide)
+    )
+    (property "Datasheet" "~" (at 118.11 83.82 0)
+      (effects (font (size 1.27 1.27)) hide)
+    )
+    (pin "1")
+    (instances
+      (project "Locator_FPGA"
+        (path "/33cb5046-a12e-4461-8dbd-367869bd8ded"
+          (reference "J13") (unit 1)
+        )
+      )
