File: Acquisition/Schematics/MIC_Extension/MIC_Extension.kicad_pcb (KiCad board)
At the start: 4 copper layers, 21.1 x 19.1 mm, 35 parts, among them J1 Conn_01x04_Pin, U1 TPS7A2033, U2 OPA188xxDBV, U5 OPA188xxDBV

Commit message: PCBs production ready
Parts:
- added C13: 10u, Capacitor_SMD:C_0603_1608Metric, F.Cu at (35.2, 65.0)
Routing:
- net Earth: track 15.5 -> 17.1 mm
- net /VddIN: track 14.9 -> 16.5 mm
Other:
- board text added: "3.3v"
- board text added: "5v"
- board text added: "GO NUTS"
- board text added: "in"
- board text added: "out"
Changed lines of the file:
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@@
     (pad_to_mask_clearance 0)
     (pcbplotparams
-      (layerselection 0x00010c0_ffffffff)
+      (layerselection 0x60010c0_ffffffff)
       (plot_on_all_layers_selection 0x0000000_00000000)
       (disableapertmacros false)
@@
       (drillshape 0)
       (scaleselection 1)
-      (outputdirectory "")
+      (outputdirectory "Gerbers/")
     )
   )
@@
   )
   (footprint "Capacitor_SMD:C_0603_1608Metric" (layer "F.Cu")
+    (at 35.179 65.037 90)
+    (descr "Capacitor SMD 0603 (1608 Metric), square (rectangular) end terminal, IPC_7351 nominal, (Body size source: IPC-SM-782 page 76, https://www.pcb-3d.com/wordpress/wp-content/uploads/ipc-sm-782a_amendment_1_and_2.pdf), generated with kicad-footprint-generator")
+    (tags "capacitor")
+    (property "Sheetfile" "MIC_Extension.kicad_sch")
+    (property "Sheetname" "")
+    (property "ki_description" "Unpolarized capacitor")
+    (property "ki_keywords" "cap capacitor")
+    (attr smd)
+    (fp_text reference "C13" (at 0 -1.43 90) (layer "F.SilkS")
+        (effects (font (size 1 1) (thickness 0.15)))
+    )
+    (fp_text value "10u" (at 0 1.43 90) (layer "F.Fab")
+        (effects (font (size 1 1) (thickness 0.15)))
+    )
+    (fp_text user "${REFERENCE}" (at 0 0 90) (layer "F.Fab")
+        (effects (font (size 0.4 0.4) (thickness 0.06)))
+    )
+    (fp_line (start -0.14058 -0.51) (end 0.14058 -0.51)
+      (stroke (width 0.12) (type solid)) (layer "F.SilkS"))
+    (fp_line (start -0.14058 0.51) (end 0.14058 0.51)
+      (stroke (width 0.12) (type solid)) (layer "F.SilkS"))
+    (fp_line (start -1.48 -0.73) (end 1.48 -0.73)
+      (stroke (width 0.05) (type solid)) (layer "F.CrtYd"))
+    (fp_line (start -1.48 0.73) (end -1.48 -0.73)
+      (stroke (width 0.05) (type solid)) (layer "F.CrtYd"))
+    (fp_line (start 1.48 -0.73) (end 1.48 0.73)
+      (stroke (width 0.05) (type solid)) (layer "F.CrtYd"))
+    (fp_line (start 1.48 0.73) (end -1.48 0.73)
+      (stroke (width 0.05) (type solid)) (layer "F.CrtYd"))
+    (fp_line (start -0.8 -0.4) (end 0.8 -0.4)
+      (stroke (width 0.1) (type solid)) (layer "F.Fab"))
+    (fp_line (start -0.8 0.4) (end -0.8 -0.4)
+      (stroke (width 0.1) (type solid)) (layer "F.Fab"))
+    (fp_line (start 0.8 -0.4) (end 0.8 0.4)
+      (stroke (width 0.1) (type solid)) (layer "F.Fab"))
+    (fp_line (start 0.8 0.4) (end -0.8 0.4)
+      (stroke (width 0.1) (type solid)) (layer "F.Fab"))
+    (pad "1" smd roundrect (at -0.775 0 90) (size 0.9 0.95) (layers "F.Cu" "F.Paste" "F.Mask") (roundrect_rratio 0.25)
+      (net 18 "/VddIN") (pintype "passive"))
+    (pad "2" smd roundrect (at 0.775 0 90) (size 0.9 0.95) (layers "F.Cu" "F.Paste" "F.Mask") (roundrect_rratio 0.25)
+      (net 1 "Earth") (pintype "passive"))
+    (model "${KICAD6_3DMODEL_DIR}/Capacitor_SMD.3dshapes/C_0603_1608Metric.wrl"
+      (offset (xyz 0 0 0))
+      (scale (xyz 1 1 1))
+      (rotate (xyz 0 0 0))
+    )
+  )
+  (footprint "Capacitor_SMD:C_0603_1608Metric" (layer "F.Cu")
     (at 36.8225 52.832)
     (descr "Capacitor SMD 0603 (1608 Metric), square (rectangular) end terminal, IPC_7351 nominal, (Body size source: IPC-SM-782 page 76, https://www.pcb-3d.com/wordpress/wp-content/uploads/ipc-sm-782a_amendment_1_and_2.pdf), generated with kicad-footprint-generator")
@@
   (gr_rect (start 32.766 48.26) (end 53.848 67.31)
     (stroke (width 0.1) (type default)) (fill none) (layer "Edge.Cuts"))
+  (gr_rect (start 48.133 55.245) (end 49.911 58.801)
+    (stroke (width 0.15) (type default)) (fill none) (layer "User.8"))
+  (gr_rect (start 43.815 60.071) (end 45.466 63.373)
+    (stroke (width 0.15) (type default)) (fill none) (layer "User.8"))
+  (gr_rect (start 47.625 48.514) (end 51.054 55.753)
+    (stroke (width 0.15) (type default)) (fill none) (layer "User.9"))
+  (gr_text "in" (at 51.435 54.483 90) (layer "User.8")
+    (effects (font (size 1 1) (thickness 0.15)) (justify left bottom mirror))
+  )
+  (gr_text "out" (at 43.307 61.087 90) (layer "User.8")
+    (effects (font (size 1 1) (thickness 0.15)) (justify left bottom mirror))
+  )
+  (gr_text "5v" (at 50.419 64.897) (layer "User.9")
+    (effects (font (size 1 1) (thickness 0.15)) (justify left bottom))
+  )
+  (gr_text "GO NUTS" (at 52.578 55.499 90) (layer "User.9")
+    (effects (font (size 1 1) (thickness 0.15)) (justify left bottom))
+  )
+  (gr_text "3.3v" (at 50.419 66.548) (layer "User.9")
+    (effects (font (size 1 1) (thickness 0.15)) (justify left bottom))
+  )
   (via (at 34.798 58.42) (size 2.5) (drill 1.8) (layers "F.Cu" "B.Cu") (net 0))
   (via (at 51.816 58.42) (size 2.5) (drill 1.8) (layers "F.Cu" "B.Cu") (net 0))
@@
   (segment (start 41.224 51.563) (end 40.386 50.725) (width 0.25) (layer "F.Cu") (net 1))
   (segment (start 43.897 62.174) (end 43.46 62.611) (width 0.25) (layer "F.Cu") (net 1))
+  (segment (start 36.817 64.262) (end 36.83 64.249) (width 0.25) (layer "F.Cu") (net 1))
   (segment (start 36.83 64.249) (end 36.83 64.389) (width 0.25) (layer "F.Cu") (net 1))
   (segment (start 37.5975 51.308) (end 37.5975 52.832) (width 0.25) (layer "F.Cu") (net 1))
@@
   (segment (start 45.105251 59.436) (end 44.979 59.309749) (width 0.25) (layer "F.Cu") (net 1))
   (segment (start 41.224 51.977) (end 41.224 51.563) (width 0.25) (layer "F.Cu") (net 1))
+  (segment (start 35.179 64.262) (end 36.817 64.262) (width 0.25) (layer "F.Cu") (net 1))
   (segment (start 49.276 54.076) (end 48.488 54.864) (width 0.25) (layer "F.Cu") (net 1))
   (via (at 50.038 49.276) (size 0.8) (drill 0.4) (layers "F.Cu" "B.Cu") (net 1))
@@
   (segment (start 49.877999 52.197) (end 50.226 52.545001) (width 0.25) (layer "F.Cu") (net 17))
   (segment (start 48.326 52.545001) (end 48.674001 52.197) (width 0.25) (layer "F.Cu") (net 17))
+  (segment (start 35.179 65.812) (end 36.817 65.812) (width 0.25) (layer "F.Cu") (net 18))
   (segment (start 39.624 66.548) (end 38.872 65.796) (width 0.5) (layer "F.Cu") (net 18))
   (segment (start 47.739 66.548) (end 39.624 66.548) (width 0.5) (layer "F.Cu") (net 18))
   (segment (start 36.83 65.799) (end 38.138 65.799) (width 0.25) (layer "F.Cu") (net 18))
   (segment (start 38.872 65.796) (end 38.872 65.065) (width 0.5) (layer "F.Cu") (net 18))
+  (segment (start 36.817 65.812) (end 36.83 65.799) (width 0.25) (layer "F.Cu") (net 18))
   (segment (start 48.501 65.786) (end 48.501 64.262) (width 0.5) (layer "F.Cu") (net 18))
   (segment (start 48.501 65.786) (end 47.739 66.548) (width 0.5) (layer "F.Cu") (net 18))
