File: Acquisition/Schematics/MIC_Extension/MIC_Extension.kicad_sch (KiCad schematic)
At the start: 35 parts, among them J1 Conn_01x04_Pin, U1 TPS7A2033, U2 OPA188xxDBV, U5 OPA188xxDBV

Commit message: PCBs production ready
Parts:
- added C13: 10u, Capacitor_SMD:C_0603_1608Metric, symbol Device:C
Connections:
- net Earth: now also C13.2
- net VddIN: now also C13.1
Changed lines of the file:
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@@
   (junction (at 62.23 45.72) (diameter 0) (color 0 0 0 0)
   )
+  (junction (at 115.57 109.22) (diameter 0) (color 0 0 0 0)
+  )
   (junction (at 132.08 167.64) (diameter 0) (color 0 0 0 0)
   )
@@
     (stroke (width 0) (type default))
   )
+  (wire (pts (xy 110.49 109.22) (xy 115.57 109.22))
+    (stroke (width 0) (type default))
+  )
   (wire (pts (xy 57.15 172.72) (xy 73.66 172.72))
     (stroke (width 0) (type default))
@@
   )
   (wire (pts (xy 134.62 50.8) (xy 135.89 50.8))
+    (stroke (width 0) (type default))
+  )
+  (wire (pts (xy 110.49 101.6) (xy 115.57 101.6))
     (stroke (width 0) (type default))
   )
@@
         )
       )
+    )
+  )
+  (symbol (lib_id "Device:C") (at 110.49 105.41 0) (unit 1)
+    (in_bom yes) (on_board yes) (dnp no) (fields_autoplaced)
+    (property "Reference" "C13" (at 114.3 104.14 0)
+      (effects (font (size 1.27 1.27)) (justify left))
+    )
+    (property "Value" "10u" (at 114.3 106.68 0)
+      (effects (font (size 1.27 1.27)) (justify left))
+    )
+    (property "Footprint" "Capacitor_SMD:C_0603_1608Metric" (at 111.4552 109.22 0)
+      (effects (font (size 1.27 1.27)) hide)
+    )
+    (property "Datasheet" "~" (at 110.49 105.41 0)
+      (effects (font (size 1.27 1.27)) hide)
+    )
+    (pin "1")
+    (pin "2")
+    (instances
+      (project "MIC_Extension"
+        (path "/8c348a62-ef66-40bd-93f1-5fbc22cdd0f1"
+          (reference "C13") (unit 1)
+        )
+      )
